Commit message: gazebo: objects world (box 33x22x11 cm + RGB 3 cm cubes); robot meshes, floor height, LiDAR self-hit
- map_to_world.py --object X Y SX SY SZ R G B MASS (coloured, dynamic when mass > 0);
  worlds/room_lap2_objects.sdf: box at (1.21, 1.00), cubes R/G/B at y 0.62 in front of start A
- sim.launch.py: add jetrover_description to GZ_SIM_RESOURCE_PATH - the robot body meshes were
  never found (70 errors), the robot was invisible and had no body collision
- room_assets.py: shift the scanned floor (z 0.044 m) to 0; visual keeps the floor (+3 mm),
  collision drops it so 3 cm cubes are not buried
- sim xacro: rear black shell hidden from the LiDAR only (visibility mask); it gave 0.16-0.27 m
  hits while the real LiDAR has no return in that sector
- host checks: objects settle, LiDAR no beams < 0.3 m, drive OK; jetrover_gazebo lint clean

File: src/jetrover_gazebo/urdf/jetrover_sim.urdf.xacro (robot description, xacro)
@@ -68,6 +68,13 @@
   <xacro:mecanum_friction link="wheel_left_back_link" fdir="1 1 0"/>
   <xacro:mecanum_friction link="wheel_right_back_link" fdir="1 -1 0"/>
-  <!-- RPLIDAR A1M8-like: 360 deg, ~10 Hz, 0.15-12 m. Frame = lidar_frame like the real driver; the arm geometry
-       occludes the rear by itself. / 실기와 같은 프레임, 팔이 뒤쪽을 실제처럼 가린다. -->
+  <!-- RPLIDAR A1M8-like: 360 deg, ~10 Hz, 0.15-12 m. Frame = lidar_frame like the real driver.
+       The rear black shell crosses the LiDAR plane: in sim it returned 0.16-0.27 m hits (lidar-frame +-12..25 deg)
+       while the real LiDAR has NO return there (0 % finite, tol015 bags, 2026-10-14). Visibility bit 0x2 hides the
+       shell from the LiDAR only (GUI/cameras still see it); the sim then sees past it - real is blind there.
+       한글: 실기와 같은 프레임. 뒤쪽 검은 덮개가 LiDAR 높이를 가로질러 시뮬레이션에서만 0.16~0.27 m로 잡혔다(실기는 그 구간 값 없음).
+       덮개를 LiDAR에서만 안 보이게(visibility 0x2) — 남는 차이: 시뮬레이션은 그 너머를 본다. -->
+  <gazebo reference="back_shell_black_link">
+    <visual><visibility_flags>2</visibility_flags></visual>
+  </gazebo>
   <gazebo reference="lidar_frame">
     <sensor name="lidar" type="gpu_lidar">
@@ -82,4 +89,5 @@
         <range><min>0.15</min><max>12.0</max><resolution>0.01</resolution></range>
         <noise><type>gaussian</type><mean>0.0</mean><stddev>0.01</stddev></noise>
+        <visibility_mask>4294967293</visibility_mask>
       </lidar>
     </sensor>

Commit message: gazebo: sim gripper mimic joints via ros2_control; pick-and-lift check 3/3
- DART has no mimic constraint, so only r_joint moved and the 5 finger joints dangled; they are now
  ros2_control state-only joints and gz_ros2_control drives them from r_joint (multiplier +-1)
- tools/sim/arm_ik.py (numeric IK on the sim URDF, gripper down) and sim_pick_check.sh/.py:
  arm-test spawn, open, descend, close r_joint 0.3, lift; red/green/blue all lifted to z 0.128 m,
  r_joint stalls at 0.34 on contact; drive from A and LiDAR unchanged

File: src/jetrover_gazebo/urdf/jetrover_sim.urdf.xacro (robot description, xacro)
@@ -40,4 +40,19 @@
     <xacro:arm_if joint="joint5" init="${home[4]}"/>
     <xacro:arm_if joint="r_joint" init="${home[5]}"/>
+    <!-- 그리퍼 연동 관절(URDF mimic): DART는 mimic 제약을 지원하지 않아 r_joint만 움직이고 손가락이 덜렁거렸다(2026-10-14).
+         상태 인터페이스만 두면 gz_ros2_control이 mimic(배율 ±1)대로 위치를 맞춘다(공식 gripper_mimic_joint_example 방식).
+         Gripper mimic joints: DART has no mimic constraint, so list them with state interfaces only and
+         gz_ros2_control drives them from r_joint (as in gz_ros2_control_demos gripper_mimic_joint_example). -->
+    <xacro:macro name="mimic_if" params="joint">
+      <joint name="${joint}">
+        <state_interface name="position"/>
+        <state_interface name="velocity"/>
+      </joint>
+    </xacro:macro>
+    <xacro:mimic_if joint="l_joint"/>
+    <xacro:mimic_if joint="l_in_joint"/>
+    <xacro:mimic_if joint="l_out_joint"/>
+    <xacro:mimic_if joint="r_in_joint"/>
+    <xacro:mimic_if joint="r_out_joint"/>
   </ros2_control>
   <gazebo>
