Commit message: Add jetrover_gazebo: Gazebo Harmonic sim with gz_ros2_control mecanum drive
- jetrover_description: sim_mode xacro arg (default false output identical to before);
  true makes the 4 wheels continuous (y axis) with sphere collisions
- jetrover_sim.urdf.xacro: ros2_control (wheel velocity, arm/gripper position held at the home
  pose), mecanum emulation as in gz_ros2_control_demos (anisotropic friction along the roller
  diagonal), gpu_lidar /scan, rgbd_camera (640x360, fx 362.5), imu
- mecanum_drive_controller (r 0.0485, lx+ly 0.2096 like base.yaml), bridge, EKF on controller
  odometry; helpers: cmd_vel Twist -> TwistStamped, depth 32FC1 m -> 16UC1 mm, arm hold
- map_to_world.py: SLAM map occupied cells -> 167 wall boxes (map frame = world frame), worlds
  with/without the test box
- Nav2/localization launches take use_sim_time; capture_depth_reference --out for a sim reference
- L0 only on the Jetson (URDF/SDF conversion, gz sdf -k, colcon test); runs on the host PC

File: src/jetrover_description/urdf/car_mecanum.urdf.xacro (robot description, xacro)
@@ -66,6 +66,11 @@
         rpy="0 0 0" />
       <geometry>
-        <mesh
-          filename="package://jetrover_description/meshes/mecanum/wheel_left_front_link_collision.stl" />
+        <xacro:if value="${sim_mode}">
+          <sphere radius="0.0485"/>  <!-- Gazebo mecanum emulation (anisotropic friction) / 시뮬 메카넘용 구 -->
+        </xacro:if>
+        <xacro:unless value="${sim_mode}">
+          <mesh
+            filename="package://jetrover_description/meshes/mecanum/wheel_left_front_link_collision.stl" />
+        </xacro:unless>
       </geometry>
     </collision>
@@ -73,5 +78,5 @@
   <joint
     name="wheel_left_front_joint"
-    type="fixed">
+    type="${'continuous' if sim_mode else 'fixed'}">
     <origin
       xyz="0.0975130769499663 0.11212949984639 -0.0678410821576751"
@@ -82,5 +87,5 @@
       link="wheel_left_front_link" />
     <axis
-      xyz="0 0 0" />
+      xyz="${'0 1 0' if sim_mode else '0 0 0'}" />
   </joint>
   <link
@@ -115,6 +120,11 @@
         rpy="0 0 0" />
       <geometry>
-        <mesh
-          filename="package://jetrover_description/meshes/mecanum/wheel_left_back_link_collision.stl" />
+        <xacro:if value="${sim_mode}">
+          <sphere radius="0.0485"/>  <!-- Gazebo mecanum emulation (anisotropic friction) / 시뮬 메카넘용 구 -->
+        </xacro:if>
+        <xacro:unless value="${sim_mode}">
+          <mesh
+            filename="package://jetrover_description/meshes/mecanum/wheel_left_back_link_collision.stl" />
+        </xacro:unless>
       </geometry>
     </collision>
@@ -122,5 +132,5 @@
   <joint
     name="wheel_left_back_joint"
-    type="fixed">
+    type="${'continuous' if sim_mode else 'fixed'}">
     <origin
       xyz="-0.0975130776687404 0.112129499199832 -0.0678410821576746"
@@ -131,5 +141,5 @@
       link="wheel_left_back_link" />
     <axis
-      xyz="0 0 0" />
+      xyz="${'0 1 0' if sim_mode else '0 0 0'}" />
   </joint>
   <link
@@ -164,6 +174,11 @@
         rpy="0 0 0" />
       <geometry>
-        <mesh
+        <xacro:if value="${sim_mode}">
+          <sphere radius="0.0485"/>  <!-- Gazebo mecanum emulation (anisotropic friction) / 시뮬 메카넘용 구 -->
+        </xacro:if>
+        <xacro:unless value="${sim_mode}">
+          <mesh
             filename="package://jetrover_description/meshes/mecanum/wheel_right_front_link_collision.stl" />
+        </xacro:unless>
       </geometry>
     </collision>
@@ -171,5 +186,5 @@
   <joint
     name="wheel_right_front_joint"
-    type="fixed">
+    type="${'continuous' if sim_mode else 'fixed'}">
     <origin
       xyz="0.0975130776687398 -0.112129499199832 -0.0678410821576747"
@@ -180,5 +195,5 @@
       link="wheel_right_front_link" />
     <axis
-      xyz="0 0 0" />
+      xyz="${'0 1 0' if sim_mode else '0 0 0'}" />
   </joint>
   <link
@@ -213,6 +228,11 @@
         rpy="0 0 0" />
       <geometry>
-        <mesh
+        <xacro:if value="${sim_mode}">
+          <sphere radius="0.0485"/>  <!-- Gazebo mecanum emulation (anisotropic friction) / 시뮬 메카넘용 구 -->
+        </xacro:if>
+        <xacro:unless value="${sim_mode}">
+          <mesh
             filename="package://jetrover_description/meshes/mecanum/wheel_right_back_link_collision.stl" />
+        </xacro:unless>
       </geometry>
     </collision>
@@ -220,5 +240,5 @@
   <joint
     name="wheel_right_back_joint"
-    type="fixed">
+    type="${'continuous' if sim_mode else 'fixed'}">
     <origin
       xyz="-0.097513076949967 -0.11212949984639 -0.0678410821576744"
@@ -229,5 +249,5 @@
       link="wheel_right_back_link" />
     <axis
-      xyz="0 0 0" />
+      xyz="${'0 1 0' if sim_mode else '0 0 0'}" />
   </joint>
 </robot>

File: src/jetrover_description/urdf/jetrover.xacro (robot description, xacro)
@@ -3,4 +3,9 @@
     <xacro:property name="lidar"        value="$(optenv LIDAR_TYPE A1)"/>
     <xacro:property name="machine"      value="$(optenv MACHINE_TYPE JetRover_Mecanum)"/>
+    <!-- sim_mode (2026-10-09, prd/gazebo-sim.md): true only for Gazebo (jetrover_gazebo). Wheels become continuous joints with
+         sphere collisions there; false (default) keeps the real-robot description unchanged (fixed wheels, mesh collisions).
+         한글: Gazebo에서만 true. 바퀴를 회전 관절+구 충돌로. 기본 false는 실기 설명 그대로. -->
+    <xacro:arg name="sim_mode" default="false"/>
+    <xacro:property name="sim_mode" value="$(arg sim_mode)"/>
     <xacro:include filename="$(find jetrover_description)/urdf/materials.xacro"/>
     <xacro:include filename="$(find jetrover_description)/urdf/inertial_matrix.xacro" />

Commit message: sim avoidance (wip): harness, metrics, precise approach node, simulation fixes
- tools/sim: avoid_trials.py (S1/S2/S4 runner with Gazebo ground truth, costmap clear per trial),
  avoid_metrics.py + tests, sim_avoid_run.sh, gt_localization.py, plant_response.py and diagnostics
- jetrover_navigation: precise_approach.py (mecanum final approach action, 8 unit tests);
  nav2.launch.py use_sim_time rewrites the params file (all nodes ran on wall time) and sim-only depth min height
- Gazebo: fdir1 frame base_footprint (strafing was wrong, troubleshooting/047), cylinder wheels of the real
  size, depth margin 100 mm and extrusion 0.25 m in the scanned room
- Nav2 variants in tools/nav/ab_params (padding, goal tolerance, ObstacleFootprint critic)

File: src/jetrover_description/urdf/car_mecanum.urdf.xacro (robot description, xacro)
@@ -63,9 +63,9 @@
     <collision>
       <origin
-        xyz="0 0 0"
-        rpy="0 0 0" />
-      <geometry>
-        <xacro:if value="${sim_mode}">
-          <sphere radius="0.0485"/>  <!-- Gazebo mecanum emulation (anisotropic friction) / 시뮬 메카넘용 구 -->
+        xyz="0 ${-0.0066 if sim_mode else 0} 0"
+        rpy="${1.5707963 if sim_mode else 0} 0 0" />
+      <geometry>
+        <xacro:if value="${sim_mode}">
+          <cylinder radius="0.0487" length="0.0488"/>  <!-- Gazebo mecanum emulation (anisotropic friction): cylinder = real wheel collision size (r 0.0487, width 0.0488, y offset as the mesh) instead of a sphere (outer edge 0.161 m vs the real 0.130 m: the simulated robot was 6 cm wider than the real one, 2026-10-19) / 시뮬 메카넘용 원통: 실기 바퀴와 같은 크기(구는 바깥 16.1 cm라 실기 13.0 cm보다 6 cm 넓었다) -->
         </xacro:if>
         <xacro:unless value="${sim_mode}">
@@ -117,9 +117,9 @@
     <collision>
       <origin
-        xyz="0 0 0"
-        rpy="0 0 0" />
-      <geometry>
-        <xacro:if value="${sim_mode}">
-          <sphere radius="0.0485"/>  <!-- Gazebo mecanum emulation (anisotropic friction) / 시뮬 메카넘용 구 -->
+        xyz="0 ${-0.0066 if sim_mode else 0} 0"
+        rpy="${1.5707963 if sim_mode else 0} 0 0" />
+      <geometry>
+        <xacro:if value="${sim_mode}">
+          <cylinder radius="0.0487" length="0.0488"/>  <!-- Gazebo mecanum emulation (anisotropic friction): cylinder = real wheel collision size (r 0.0487, width 0.0488, y offset as the mesh) instead of a sphere (outer edge 0.161 m vs the real 0.130 m: the simulated robot was 6 cm wider than the real one, 2026-10-19) / 시뮬 메카넘용 원통: 실기 바퀴와 같은 크기(구는 바깥 16.1 cm라 실기 13.0 cm보다 6 cm 넓었다) -->
         </xacro:if>
         <xacro:unless value="${sim_mode}">
@@ -171,9 +171,9 @@
     <collision>
       <origin
-        xyz="0 0 0"
-        rpy="0 0 0" />
-      <geometry>
-        <xacro:if value="${sim_mode}">
-          <sphere radius="0.0485"/>  <!-- Gazebo mecanum emulation (anisotropic friction) / 시뮬 메카넘용 구 -->
+        xyz="0 ${0.0066 if sim_mode else 0} 0"
+        rpy="${1.5707963 if sim_mode else 0} 0 0" />
+      <geometry>
+        <xacro:if value="${sim_mode}">
+          <cylinder radius="0.0487" length="0.0488"/>  <!-- Gazebo mecanum emulation (anisotropic friction): cylinder = real wheel collision size (r 0.0487, width 0.0488, y offset as the mesh) instead of a sphere (outer edge 0.161 m vs the real 0.130 m: the simulated robot was 6 cm wider than the real one, 2026-10-19) / 시뮬 메카넘용 원통: 실기 바퀴와 같은 크기(구는 바깥 16.1 cm라 실기 13.0 cm보다 6 cm 넓었다) -->
         </xacro:if>
         <xacro:unless value="${sim_mode}">
@@ -225,9 +225,9 @@
     <collision>
       <origin
-        xyz="0 0 0"
-        rpy="0 0 0" />
-      <geometry>
-        <xacro:if value="${sim_mode}">
-          <sphere radius="0.0485"/>  <!-- Gazebo mecanum emulation (anisotropic friction) / 시뮬 메카넘용 구 -->
+        xyz="0 ${0.0066 if sim_mode else 0} 0"
+        rpy="${1.5707963 if sim_mode else 0} 0 0" />
+      <geometry>
+        <xacro:if value="${sim_mode}">
+          <cylinder radius="0.0487" length="0.0488"/>  <!-- Gazebo mecanum emulation (anisotropic friction): cylinder = real wheel collision size (r 0.0487, width 0.0488, y offset as the mesh) instead of a sphere (outer edge 0.161 m vs the real 0.130 m: the simulated robot was 6 cm wider than the real one, 2026-10-19) / 시뮬 메카넘용 원통: 실기 바퀴와 같은 크기(구는 바깥 16.1 cm라 실기 13.0 cm보다 6 cm 넓었다) -->
         </xacro:if>
         <xacro:unless value="${sim_mode}">

File: src/jetrover_gazebo/urdf/jetrover_sim.urdf.xacro (robot description, xacro)
@@ -63,7 +63,12 @@
     </plugin>
   </gazebo>
-  <!-- Mecanum emulation exactly as gz_ros2_control_demos test_mecanum_drive: friction only along the roller
-       diagonal (fdir1, in base_link), none across it (mu2 = 0). X pattern seen from above; verify by strafing on host.
-       한글: 공식 데모와 같은 방식. 롤러 대각 방향으로만 마찰. 위에서 X자 배치 — host에서 옆이동 방향으로 확인. -->
+  <!-- Mecanum emulation as gz_ros2_control_demos test_mecanum_drive: friction only along the roller diagonal (fdir1),
+       none across it (mu2 = 0). X pattern seen from above.
+       fdir1 is expressed in base_footprint, NOT base_link (2026-10-19, troubleshooting/047): base_link is lumped into
+       base_footprint by the fixed joint, so DART found no body node ("Failed to get body node for [wheel_*_collision], not
+       setting friction direction frame") and the roller direction rotated with the spinning wheel: strafing went the wrong
+       way and diagonals turned the robot. Measured with tools/sim/plant_response.py after the fix: strafe, diagonal and
+       rotation ratios 1.00 with no cross components.
+       한글: 공식 데모와 같은 방식. fdir1 기준 프레임은 base_link가 아니라 base_footprint다(base_link는 fixed joint로 합쳐져 없음). -->
   <xacro:macro name="mecanum_friction" params="link fdir">
     <gazebo reference="${link}">
@@ -74,5 +79,5 @@
               <mu>1.0</mu>
               <mu2>0.0</mu2>
-              <fdir1 gz:expressed_in="base_link">${fdir}</fdir1>
+              <fdir1 gz:expressed_in="base_footprint">${fdir}</fdir1>
             </ode>
           </friction>
